File: KiCAD/Projeto SEMB.kicad_sch (KiCad schematic)
At the start: 58 parts, among them J2 ST-Link V2, M1 Motor_DC, M2 Motor_DC, Q1 IRLML5203, Q2 IRLML5203, SW1 Reset, SW2 BOOT_0, U1 STM32F411CEUx, U2 2SMPP-03, U3 TLV2371P, U4 DRV8212P, U5 TPS7A2433DBVR, U6 TLV2371P, U7 4N25, U8 TLV2371P, U9 TLV2371P, Y1 LSE, Y2 HSE

Commit message: Correção  Sensor de Pressão KiCAD
Parts:
- removed U2: 2SMPP-03, 2SMPP-03_OMR, symbol 2024-09-16_13-36-37:2SMPP-03
- added C18, C20, C21: 105uF, symbol Device:C
- added C19: 330uF, symbol Device:C_Polarized
- added C22: 220uF, symbol Device:C_Polarized
- added D5: BZV55B43, Diode_SMD:D_MiniMELF, symbol Diode:BZV55B43
- added J1: Battery-12V, symbol Connector_Generic:Conn_01x02
- added L3: 47uH, symbol Device:L
- added R18, R20: 10k, symbol Device:R
- added R19: 3.3k, symbol Device:R
- added U10: XL4015, Package_TO_SOT_SMD:TO-263-5_TabPin3, symbol Regulator_Switching:XL4015
- added U2: 2SMPP-03, 2SMPP-03_OMR, symbol 2SMPP03:2SMPP-03
- R10, R11, R13, R14, R15, R16, R17: value R -> 10k
- R12: value R -> 1k
- R9: value R -> 40k
Connections:
- net +11V is gone; now on net +5V: C7.1, U5.1 (IN), U5.3 (EN)
- net 3.3V: no longer R9.1
- net GND: now also U3.4 (V-), U6.4 (V-), U8.7 (V+), U9.7 (V+), C18.2, C19.2, C21.2, C22.2, D5.2 (A), J1.1 (Pin_1), R19.2, R20.2, U10.1 (GND)
- net at U8.3 (+): now also U2.4 (VOUT-)
- net +5V: now reaches U8.4 (V-)
- net +5V: now also R9.1, U3.7 (V+), U6.7 (V+), U9.4 (V-), C18.1, C19.1, L3.2, R18.1
- net at U6.3 (+): now also U2.1 (VOUT+)
- net at U3.6: now also U2.5 (N-SUB), U2.6 (ICC)
- new net: C20.1, C21.1, C22.1, J1.2 (Pin_2), U10.5 (VIN)
- new net: C20.2, U10.4 (VC)
- new net: R18.2, R19.1, U10.2 (FB)
- new net: R20.1, U2.3 (GND)
- new net: D5.1 (K), L3.1, U10.3 (SW)
- no-connect marks 0 -> 28
Other:
- note added: "0V - 0.651V"
- note added: "DC-DC Step-Down +12V to +5V"
- note added: "DC-DC Step-Down +5V to +3.3V"
- note added: "Output 0 mV ~ 31 mV"
- note added: "V1"
- note added: "V2"
- note added: "VOUT = (1+2R2/R1)*(V2-V1)"
- note added: "VOUT = 1.25*(1+R2/R1)"
- note removed: "DC-DC Step-Down +12V to +3.3V"
- moved on the sheet: C3, C4, C5, C6, C7, D1, M1, M2, Q1, R3, R6, R7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

Commit message: Mudanças no Esquemático -> Priorização do Circuito com Driver do Motor DC e Correção dos Warnings do Electrical Rule Checker
Parts:
- removed D1: 1N4148, Diode_THT:D_DO-35_SOD27_P7.62mm_Horizontal, symbol Diode:1N4148
- removed M2: Motor_DC, symbol Motor:Motor_DC
- removed Q1: IRLML5203, Package_TO_SOT_SMD:SOT-23, symbol Transistor_FET:IRLML5203
- removed R3: 1k, symbol Device:R
- removed U5: TPS7A2433DBVR, SOT23_DBV_TEX, symbol 2024-09-16_13-49-55:TPS7A2433DBVR
- removed U7: 4N25, Package_DIP:DIP-6_W7.62mm, symbol Isolator:4N25
- added U7: TPS7A2433DBVR, SOT23_DBV_TEX, symbol TPS7A2433DBVR:TPS7A2433DBVR
- L2: value L -> 1mH
Connections:
- net +12V: now also C20.1, C21.1, C22.1, J1.2 (Pin_2), U10.5 (VIN)
- net +3.3V: now also U7.5 (OUT)
- net +5V: now also U7.1 (IN), U7.3 (EN)
- net GND: now also U7.2 (GND)
- net PC14: no longer C14.1, U1.4 (PC15), Y1.2
- net PH0: no longer C17.1, U1.6 (PH1), Y2.2
- net at R6.2, R7.1: now also U7.4 (FB)
- new net PC15: C14.1, U1.4 (PC15), Y1.2
- new net PH1: C17.1, U1.6 (PH1), Y2.2
- no-connect marks 28 -> 27
Other:
- note added: "Display & User Interface"
- note added: "GND"
- note added: "HSE(+)"
- note added: "HSE(-)"
- note added: "IN1"
- note added: "IN2"
- note added: "LSE(+)"
- note added: "LSE(-)"
- note added: "Pression"
- note added: "SWCLK"
- note added: "SWDIO"
- note added: "Valve"
- note removed: "Alternative Motor Circuit"

Commit message: Atualização de Datasheets e inclusão do LCD com expansor I²C
Parts:
- added RV1: R_Potentiometer_Trim, symbol Device:R_Potentiometer_Trim
- added SW3: SW_SPDT, symbol Switch:SW_SPDT
- added U11: LCD-016N002L, Display:LCD-016N002L, symbol Display_Character:LCD-016N002L
- added U5: PCF8574A, symbol Interface_Expansion:PCF8574A
Connections:
- net +12V: now also SW3.3 (C); no longer C20.1, C21.1, C22.1, U10.5 (VIN)
- net +5V: now also U11.15 (A/VEE), U11.2 (VDD), U11.A1, U11.A2, U5.13 (~{INT}), U5.16 (VDD)
- net 3.3V: now also RV1.3
- net GND: now also RV1.1, SW3.1 (A), U11.1 (VSS), U11.16 (K), U11.5 (R/~{W}), U11.K1, U11.K2, U5.1 (A0), U5.2 (A1), U5.3 (A2), U5.8 (VSS)
- net PB14: now reaches U1.27 (PB14)
- net PB14: now also R16.1, U9.6
- net PB4: now reaches U1.40 (PB4)
- net PB4: now also U11.4 (RS)
- net PB5: now reaches U1.41 (PB5)
- net PB5: now also U11.6 (E)
- net PB6: now reaches U1.42 (PB6)
- net PB6: now also U5.14 (SCL)
- net PB7: now reaches U1.43 (PB7)
- net PB7: now also U5.15 (SDA)
- removed net PB13: R16.1, U1.26 (PB13), U9.6
- new net: C20.1, C21.1, C22.1, SW3.2 (B), U10.5 (VIN)
- new net: RV1.2, U11.3 (VO)
- new net: U11.10 (DB3), U5.7 (P3)
- new net: U11.11 (DB4), U5.9 (P4)
- new net: U11.12 (DB5), U5.10 (P5)
- new net: U11.13 (DB6), U5.11 (P6)
- new net: U11.14 (DB7), U5.12 (P7)
- new net: U11.7 (DB0), U5.4 (P0)
- new net: U11.8 (DB1), U5.5 (P1)
- new net: U11.9 (DB2), U5.6 (P2)
- no-connect marks 27 -> 23
Other:
- note added: "*Especificações do Datasheet: É necessário uma fonte de corrente constante na entrada (ICC e N-Sub) A tensão de referência está conectada a um AO com saída de corrente constante"
- note added: "Contrast modulation"
- note added: "Enable"
- note added: "RS"
- note added: "SCL"
- note added: "SDA"
- moved on the sheet: C18, C19, C20, C21, C22, D5, J1, L3, R18, R19, U10

Commit message: BOM
Parts:
- added R21, R3: 4k7, Resistor_SMD:R_0603_1608Metric_Pad0.98x0.95mm_HandSolder, symbol Device:R
- added U12: TLV172IDCK, Package_TO_SOT_SMD:SOT-353_SC-70-5, symbol Amplifier_Operational:TLV172IDCK
- C1, C10, C11, C12, C13, C14, C15, C16, C17, C18, C19, C2, C20, C21, C22, C3, C4, C5, C6, C7, C8, C9: footprint (none) -> Capacitor_SMD:C_0603_1608Metric
- D3, D4: footprint (none) -> Diode_SMD:D_0201_0603Metric
- J1, L1, M1, U5: footprint (none) -> Connector_PinHeader_2.00mm:PinHeader_1x02_P2.00mm_Vertical
- J2: footprint (none) -> Connector_PinHeader_2.00mm:PinHeader_1x04_P2.00mm_Vertical
- L2, L3: footprint (none) -> Inductor_SMD:L_0603_1608Metric
- R1, R10, R14, R15, R16, R17, R18, R19, R2, R20, R4, R5, R6, R7, R8, R9: footprint (none) -> Resistor_SMD:R_0603_1608Metric_Pad0.98x0.95mm_HandSolder
- R11, R13: value 10k -> 100k; footprint (none) -> Resistor_SMD:R_0603_1608Metric_Pad0.98x0.95mm_HandSolder
- R12: value 1k -> 2k; footprint (none) -> Resistor_SMD:R_0603_1608Metric_Pad0.98x0.95mm_HandSolder
- RV1: footprint (none) -> Potentiometer_SMD:Potentiometer_Bourns_3269W_Vertical
- SW1, SW2: footprint (none) -> Button_Switch_SMD:SW_SPST_B3U-1000P-B
- SW3: footprint (none) -> Button_Switch_SMD:SW_DIP_SPSTx0l_Slide_9.78x4.72mm_W8.61mm_P2.54mm
- Y1, Y2: footprint (none) -> Crystal:Crystal_SMD_SeikoEpson_FA238V-4Pin_3.2x2.5mm
Connections:
- net +3.3V: now also U12.1 (+); no longer C10.1, C2.1, C8.1, C9.1, U1.24 (VDD), U1.36 (VDD), U1.48 (VDD), U4.7 (~{SLEEP})
- net +5V: now also U9.7 (V+), R21.1, R3.1, U12.5 (V+); no longer U5.13 (~{INT}), U9.4 (V-)
- net 3.3V: now also U4.7 (~{SLEEP})
- net GND: now also U11.4 (RS), U9.4 (V-), U12.2 (V-); no longer U9.7 (V+)
- net PB6: now also R3.2
- net PB7: now also R21.2
- net at R14.1, R17.2: now also U9.2 (-); no longer U9.3 (+)
- net at R15.1, R16.2: now also U9.3 (+); no longer U9.2 (-)
- net PB4: no longer names the net of U1.40 (PB4)
- net PB4: no longer U11.4 (RS)
- new net VDD: C10.1, C2.1, C8.1, C9.1, U1.24 (VDD), U1.36 (VDD), U1.48 (VDD), U12.3 (-), U12.4
- no-connect marks 23 -> 25
Other:
- note added: "Erro ~ +/- 5.1%"
- note added: "V1 ~ 0V"
- note added: "Vout = 0V ~ 3.3V"
- note removed: "0V - 0.651V"
- note removed: "RS"
- moved on the sheet: C10, C2, C8, C9

Commit message: PRJ2-Final
Other:
- note added: "Autoria: Stephan Costa Barros Gustavo Valle Sato Solano Jorenti Jacyntho Bruno Mendes da Silva"
Changed lines of the file:
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@@
+		)
+	)
+	(text "Autoria:\n\nStephan Costa Barros\nGustavo Valle Sato \nSolano Jorenti Jacyntho \nBruno Mendes da Silva "
+		(exclude_from_sim no)
+		(at 558.546 365.506 0)
+		(effects
+			(font
+				(size 1.27 1.27)
+			)
 		)
 	)

Commit message: Footprints
Parts:
- removed C16, C17: 12pF, Capacitor_SMD:C_0603_1608Metric, symbol Device:C
- removed R11, R13: 100k, Resistor_SMD:R_0603_1608Metric_Pad0.98x0.95mm_HandSolder, symbol Device:R
- removed R12: 2k, Resistor_SMD:R_0603_1608Metric_Pad0.98x0.95mm_HandSolder, symbol Device:R
- removed R14, R15, R16, R17: 10k, Resistor_SMD:R_0603_1608Metric_Pad0.98x0.95mm_HandSolder, symbol Device:R
- removed U12: TLV172IDCK, Package_TO_SOT_SMD:SOT-353_SC-70-5, symbol Amplifier_Operational:TLV172IDCK
- removed U6, U8, U9: TLV2371P, Package_DIP:DIP-8_W7.62mm, symbol Amplifier_Operational:TLV2371P
- removed Y2: HSE, Crystal:Crystal_SMD_SeikoEpson_FA238V-4Pin_3.2x2.5mm, symbol Device:Crystal
- added C23: 0.1uF, Capacitor_SMD:C_0603_1608Metric, symbol Device:C
- added R22: 1.01k, Resistor_SMD:R_0603_1608Metric_Pad0.98x0.95mm_HandSolder, symbol Device:R
- added U13: INA333xxDGK, Package_SO:VSSOP-8_3x3mm_P0.65mm, symbol Amplifier_Instrumentation:INA333xxDGK
- C1: footprint Capacitor_SMD:C_0603_1608Metric -> Capacitor_THT:CP_Radial_D8.0mm_P3.80mm
- SW3: footprint Button_Switch_SMD:SW_DIP_SPSTx0l_Slide_9.78x4.72mm_W8.61mm_P2.54mm -> Button_Switch_SMD:SW_SPDT_CK_JS102011SAQN
- U2: footprint 2SMPP-03_OMR -> Imported:2SMPP-03_OMR
- U5: footprint Connector_PinHeader_2.00mm:PinHeader_1x02_P2.00mm_Vertical -> Imported:SOIC127P1032X265-16N
- U7: footprint SOT23_DBV_TEX -> Imported:SOT23_DBV_TEX
Connections:
- net VDD is gone; now on net +3.3V: C10.1, C2.1, C8.1, C9.1, U1.24 (VDD), U1.36 (VDD), U1.48 (VDD)
- net +3.3V: now also C5.1, U4.8 (VCC)
- net +5V: now also U13.7 (V+)
- net 3.3V: no longer C5.1, U4.8 (VCC)
- net GND: now also C23.1, C23.2, U13.4 (V-), U13.5 (Ref)
- net PA8: now also U4.6 (IN1); no longer U4.5 (IN2)
- net PA9: now also U4.5 (IN2); no longer U4.6 (IN1)
- net PB14: now also U13.6
- net at U2.1 (VOUT+): now also U13.3 (+)
- net at U2.4 (VOUT-): now also U13.2 (-)
- new net: R22.1, U13.1 (Rg)
- new net: R22.2, U13.8 (Rg)
Other:
- note removed: "25MHz"
- note removed: "Erro ~ +/- 5.1%"
- note removed: "V1"
- note removed: "V1 ~ 0V"
- note removed: "V2"
- note removed: "VOUT = (1+2R2/R1)*(V2-V1)"
- note removed: "Vout = 0V ~ 3.3V"
- moved on the sheet: C10, C8, C9, R10, R20, R9, U2, U3

Commit message: Footprints
Parts:
- added R11: 1k, Resistor_SMD:R_0603_1608Metric_Pad0.98x0.95mm_HandSolder, symbol Device:R
- added R12: 10k, Resistor_SMD:R_0603_1608Metric_Pad0.98x0.95mm_HandSolder, symbol Device:R
- added SW4: User Button, Button_Switch_SMD:SW_SPST_B3U-1000P-B, symbol Switch:SW_Push
Connections:
- net +3.3V: now also R11.1
- net GND: now also R12.1
- net PB14: now also R12.2, SW4.2; no longer U13.6
- net PA3: now reaches U1.13 (PA3)
- net PA3: now also U13.6
- new net: R11.2, SW4.1
- no-connect marks 25 -> 24
Other:
- note added: "Button"
- moved on the sheet: R21, R3, RV1, U11, U5

Commit message: User Interface
Parts:
- added BZ1: Buzzer, Buzzer_Beeper:Buzzer_Mallory_AST1109MLTRQ, symbol Device:Buzzer
- added D1: 1N4007, Diode_THT:D_DO-41_SOD81_P10.16mm_Horizontal, symbol Diode:1N4007
- added R13: 100R, Resistor_SMD:R_0603_1608Metric_Pad0.98x0.95mm_HandSolder, symbol Device:R
Connections:
- net +5V: now also U5.13 (~{INT})
- net GND: now also BZ1.2 (-), D1.2 (A)
- net PA10: now reaches U1.31 (PA10)
- net PA10: now also R13.2
- net PH0: no longer names the net of U1.5 (PH0)
- net PH1: no longer names the net of U1.6 (PH1)
- new net: BZ1.1 (+), D1.1 (K), R13.1
Other:
- note removed: "HSE(+)"
- note removed: "HSE(-)"
- moved on the sheet: C1, C10, C11, C12, C8, C9, D3, D4, L2, R11, R12, R4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
