File: KiCAD/Projeto SEMB.kicad_sch (KiCad schematic)
At the start: 67 parts, among them J1 Battery-12V, J2 ST-Link V2, M1 Motor_DC, Q2 IRLML5203, SW1 Reset, SW2 BOOT_0, SW3 SW_SPDT, SW4 User Button, U1 STM32F411CEUx, U10 XL4015, U11 LCD-016N002L, U13 INA333xxDGK, U2 2SMPP-03, U3 TLV2371P, U4 DRV8212P, U5 PCF8574A, U7 TPS7A2433DBVR, Y1 LSE

Commit message: Atualizando esquemático
Parts:
- removed R10: 10k, Resistor_SMD:R_0603_1608Metric_Pad0.98x0.95mm_HandSolder, symbol Device:R
- removed U2: 2SMPP-03, Imported:2SMPP-03_OMR, symbol 2SMPP03:2SMPP-03
- added Q2, Q3, Q4, Q5, Q6, Q7, Q8, Q9: IRF740, Package_TO_SOT_THT:TO-220-3_Vertical, symbol Transistor_FET:IRF740
- added R13, R14, R15, R16, R17, R18, R19, R20, R21, R22, R23, R24, R25, R26, R27, R28: 10k, Resistor_SMD:R_0603_1608Metric_Pad0.98x0.95mm_HandSolder, symbol Device:R
- added U2: 2SMPP-03, Imported:2SMPP-03_OMR, symbol 2SMPP-03:2SMPP-03
- R5: renamed from R9; value 40k -> 1K
- renumbered C22 to C1, C3 to C10, C4 to C11, C8 to C12, C9 to C13, C10 to C14, C1 to C15, C11 to C16, C12 to C17, C15 to C18, C14 to C19, C13 to C20, C20 to C3, C18 to C4, C19 to C5, C23 to C6, C6 to C8, C5 to C9, D5 to D1, D1 to D3, D3 to D5, L3 to L1, L1 to L2, L2 to L3, Q2 to Q1, R18 to R1, R7 to R10, R19 to R2, R21 to R29, R1 to R3, R3 to R30, R4 to R31, R5 to R32, R8 to R33, R13 to R34, R2 to R4, R20 to R6, R22 to R7, R6 to R8
Connections:
- net +3.3V: now also R29.1, R30.1, R5.1, U13.7 (V+), U3.7 (V+), U4.7 (~{SLEEP}), U5.16 (VDD), Q2.1 (G), Q3.1 (G), Q4.1 (G), Q5.1 (G), Q6.1 (G), Q7.1 (G), Q8.1 (G), Q9.1 (G), R13.2, R15.2, R17.2, R19.2, R21.2, R23.2, R25.2, R27.2
- net +5V: now also RV1.3, R14.2, R16.2, R18.2, R20.2, R22.2, R24.2, R26.2, R28.2; no longer R29.1, R30.1, R5.1, U13.7 (V+), U3.7 (V+), U5.16 (VDD)
- net 3.3V: no longer RV1.3, U4.7 (~{SLEEP})
- net at U13.3 (+): now also U2.1 (VOUT+)
- net at R6.1: now also U2.3 (GND)
- net at U13.2 (-): now also U2.4 (VOUT-)
- net at U3.6: now also U2.5 (N-SUB), U2.6 (ICC)
- net DB3: now reaches U11.10 (DB3)
- net DB3: now also Q4.2 (D), R20.1; no longer U5.7 (P3)
- net DB4: now reaches U11.11 (DB4)
- net DB4: now also Q5.2 (D), R22.1; no longer U5.9 (P4)
- net DB5: now reaches U11.12 (DB5)
- net DB5: now also Q6.2 (D), R24.1; no longer U5.10 (P5)
- net DB6: now reaches U11.13 (DB6)
- net DB6: now also Q7.2 (D), R26.1; no longer U5.11 (P6)
- net DB7: now reaches U11.14 (DB7)
- net DB7: now also Q8.2 (D), R28.1; no longer U5.12 (P7)
- net DB0: now reaches U11.7 (DB0)
- net DB0: now also Q2.2 (D), R14.1; no longer U5.4 (P0)
- net DB1: now reaches U11.8 (DB1)
- net DB1: now also Q9.2 (D), R16.1; no longer U5.5 (P1)
- net DB2: now reaches U11.9 (DB2)
- net DB2: now also Q3.2 (D), R18.1; no longer U5.6 (P2)
- new net P0: Q2.3 (S), R13.1, U5.4 (P0)
- new net P1: Q9.3 (S), R15.1, U5.5 (P1)
- new net P2: Q3.3 (S), R17.1, U5.6 (P2)
- new net P3: Q4.3 (S), R19.1, U5.7 (P3)
- new net P4: Q5.3 (S), R21.1, U5.9 (P4)
- new net P5: Q6.3 (S), R23.1, U5.10 (P5)
- new net P6: Q7.3 (S), R25.1, U5.11 (P6)
- new net P7: Q8.3 (S), R27.1, U5.12 (P7)
Other:
- note added: "Amplificador de Instrumentação com 100 de ganho"
- note added: "Display Interface"
- note added: "Logic Level Converter Block"
- note added: "User Interface"
- note removed: "Display & User Interface"
- moved on the sheet: BZ1, C12, C13, C14, C15, C16, C17, C18, C19, C20, D3, D4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

Commit message: .
Connections:
- net GND: no longer C6.1, U13.4 (V-)
- new net: C6.1, U13.4 (V-)
Other:
- moved on the sheet: C6
Changed lines of the file:
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@@
 	)
 	(junction
-		(at 519.43 82.55)
-		(diameter 0)
-		(color 0 0 0 0)
-	)
-	(junction
 		(at 200.66 341.63)
 		(diameter 0)
@@
 	(wire
 		(pts
-			(xy 515.62 82.55) (xy 519.43 82.55)
-		)
-		(stroke
-			(width 0)
-			(type default)
-		)
-	)
-	(wire
-		(pts
 			(xy 109.22 172.72) (xy 63.5 172.72)
 		)
@@
 	(wire
 		(pts
+			(xy 519.43 81.28) (xy 519.43 87.63)
+		)
+		(stroke
+			(width 0)
+			(type default)
+		)
+	)
+	(wire
+		(pts
 			(xy 367.03 184.15) (xy 356.87 184.15)
 		)
@@
 	(wire
 		(pts
-			(xy 519.43 81.28) (xy 519.43 82.55)
-		)
-		(stroke
-			(width 0)
-			(type default)
-		)
-	)
-	(wire
-		(pts
 			(xy 492.76 295.91) (xy 501.65 295.91)
 		)
@@
 	(wire
 		(pts
-			(xy 519.43 82.55) (xy 519.43 88.9)
-		)
-		(stroke
-			(width 0)
-			(type default)
-		)
-	)
-	(wire
-		(pts
 			(xy 276.86 203.2) (xy 273.05 203.2)
 		)
@@
 	(wire
 		(pts
-			(xy 515.62 87.63) (xy 515.62 82.55)
-		)
-		(stroke
-			(width 0)
-			(type default)
-		)
-	)
-	(wire
-		(pts
 			(xy 256.54 228.6) (xy 256.54 232.41)
 		)
@@
 	(symbol
 		(lib_id "power:GND")
-		(at 515.62 95.25 0)
+		(at 519.43 95.25 0)
 		(unit 1)
 		(exclude_from_sim no)
@@
 		(fields_autoplaced yes)
 		(property "Reference" "#PWR042"
-			(at 515.62 101.6 0)
+			(at 519.43 101.6 0)
 			(effects
 				(font
@@
 		)
 		(property "Value" "GND"
-			(at 515.62 100.33 0)
+			(at 519.43 100.33 0)
 			(effects
 				(font
@@
 		)
 		(property "Footprint" ""
-			(at 515.62 95.25 0)
+			(at 519.43 95.25 0)
 			(effects
 				(font
@@
 		)
 		(property "Datasheet" ""
-			(at 515.62 95.25 0)
+			(at 519.43 95.25 0)
 			(effects
 				(font
@@
 		)
 		(property "Description" "Power symbol creates a global label with name \"GND\" , ground"
-			(at 515.62 95.25 0)
+			(at 519.43 95.25 0)
 			(effects
 				(font
@@
 	(symbol
 		(lib_id "power:GND")
-		(at 519.43 88.9 0)
-		(unit 1)
-		(exclude_from_sim no)
-		(in_bom yes)
-		(on_board yes)
-		(dnp no)
-		(fields_autoplaced yes)
-		(property "Reference" "#PWR040"
-			(at 519.43 95.25 0)
-			(effects
-				(font
-					(size 1.27 1.27)
-				)
-				(hide yes)
-			)
-		)
-		(property "Value" "GND"
-			(at 519.43 93.98 0)
-			(effects
-				(font
-					(size 1.27 1.27)
-				)
-			)
-		)
-		(property "Footprint" ""
-			(at 519.43 88.9 0)
-			(effects
-				(font
-					(size 1.27 1.27)
-				)
-				(hide yes)
-			)
-		)
-		(property "Datasheet" ""
-			(at 519.43 88.9 0)
-			(effects
-				(font
-					(size 1.27 1.27)
-				)
-				(hide yes)
-			)
-		)
-		(property "Description" "Power symbol creates a global label with name \"GND\" , ground"
-			(at 519.43 88.9 0)
-			(effects
-				(font
-					(size 1.27 1.27)
-				)
-				(hide yes)
-			)
-		)
-		(pin "1"
-		)
-		(instances
-			(project "Projeto SEMB"
-				(path "/e576cbff-e477-466e-a47a-1f1d317769d9"
-					(reference "#PWR040")
-					(unit 1)
-				)
-			)
-		)
-	)
-	(symbol
-		(lib_id "power:GND")
 		(at 521.97 81.28 0)
 		(unit 1)
@@
 	(symbol
 		(lib_id "Device:C")
-		(at 515.62 91.44 0)
+		(at 519.43 91.44 0)
 		(unit 1)
 		(exclude_from_sim no)
@@
 		(dnp no)
 		(property "Reference" "C6"
-			(at 512.064 91.694 0)
+			(at 515.874 91.694 0)
 			(effects
 				(font
@@
 		)
 		(property "Value" "0.1uF"
-			(at 512.572 93.98 0)
+			(at 516.382 93.98 0)
 			(effects
 				(font
@@
 		)
 		(property "Footprint" "Capacitor_SMD:C_0603_1608Metric"
-			(at 516.5852 95.25 0)
+			(at 520.3952 95.25 0)
 			(effects
 				(font
@@
 		)
 		(property "Datasheet" "~"
-			(at 515.62 91.44 0)
+			(at 519.43 91.44 0)
 			(effects
 				(font
@@
 		)
 		(property "Description" "Unpolarized capacitor"
-			(at 515.62 91.44 0)
+			(at 519.43 91.44 0)
 			(effects
 				(font
